Commit message: added fixed torso argument to TIAGo pro

File: tiago_pro_description/robots/tiago_pro.urdf.xacro (robot description, xacro)
@@ -35,4 +35,6 @@
 <xacro:property name="ft_sensor_right" value="$(arg ft_sensor_right)" />
 <xacro:property name="arm_model" value="tiago-pro" />
+<xacro:arg name="fixed_torso" default="false" />
+<xacro:property name="fixed_torso" value="$(arg fixed_torso)" />
 <xacro:if
   value="${end_effector_left not in ['pal-pro-gripper', 'false', False, 'custom', 'no-ee']}">

File: tiago_pro_description/urdf/torso/torso_dual.urdf.xacro (robot description, xacro)
@@ -133,18 +133,27 @@
     </collision>
   </link>
-  <joint name="${name}_lift_joint" type="prismatic">
-    <origin rpy="0.0 0.0 0.0" xyz="0.0 0.0 0.5545" />
-    <parent link="${name}_fixed_link" />
-    <child link="${name}_lift_link" />
-    <axis xyz="0 0 1" />
-    <limit effort="2000" lower="0" upper="0.35" velocity="${torso_max_vel}" />
-    <calibration rising="0.0" />
-    <dynamics damping="1000" />
-    <safety_controller k_position="20"
-                         k_velocity="20"
-                         soft_lower_limit="0.0"
-                         soft_upper_limit="0.35" />
-  </joint>
-  <xacro:torso_simple_transmission name="torso_lift" reduction="1.0"/>
+  <xacro:if value="$(arg fixed_torso)">
+    <joint name="${name}_lift_joint" type="fixed">
+      <origin rpy="0.0 0.0 0.0" xyz="0.0 0.0 0.70" />
+      <parent link="${name}_fixed_link" />
+      <child link="${name}_lift_link" />
+    </joint>
+  </xacro:if>
+  <xacro:unless value="$(arg fixed_torso)">
+    <joint name="${name}_lift_joint" type="prismatic">
+      <origin rpy="0.0 0.0 0.0" xyz="0.0 0.0 0.5545" />
+      <parent link="${name}_fixed_link" />
+      <child link="${name}_lift_link" />
+      <axis xyz="0 0 1" />
+      <limit effort="2000" lower="0" upper="0.35" velocity="${torso_max_vel}" />
+      <calibration rising="0.0" />
+      <dynamics damping="1000" />
+      <safety_controller k_position="20"
+        k_velocity="20"
+        soft_lower_limit="0.0"
+        soft_upper_limit="0.35" />
+    </joint>
+    <xacro:torso_simple_transmission name="torso_lift" reduction="1.0" />
+  </xacro:unless>
   <gazebo reference="${name}_lift_joint">
      <implicitSpringDamper>1</implicitSpringDamper>
