Commit message: fix head limits

File: tiago_pro_description/urdf/head/head.urdf.xacro (robot description, xacro)
@@ -22,6 +22,6 @@
   <xacro:property name="head_1_lower_limit" value="-55"/>
   <xacro:property name="head_1_upper_limit" value="55"/>
-  <xacro:property name="head_2_lower_limit" value="-20"/>
-  <xacro:property name="head_2_upper_limit" value="55"/>
+  <xacro:property name="head_2_lower_limit" value="-55"/>
+  <xacro:property name="head_2_upper_limit" value="20"/>
   <xacro:property name="head_eps"      value="${0.07}" />
   <xacro:property name="head_1_joint_offset"      value="${0.0}" />
